File: pin_driver_npn.kicad_sch (KiCad schematic)
At the start: 7 parts, among them Q701 BC847BS

Commit message: add mouser part numbers
Parts:
- Q701: MOUSER (none) -> 241-BC847BS_R1_00001
- R701, R702: MOUSER (none) -> 603-RC0805FR-074K7L
- R703, R704: MOUSER (none) -> 603-AC0805FR-1047KL
- R705, R706: MOUSER (none) -> 603-RC0805JR-07100KL
Changed lines of the file:
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@@
 			)
 		)
-		(property "MOUSER" ""
+		(property "MOUSER" "603-AC0805FR-1047KL"
 			(at 204.47 86.36 90)
+			(effects
+				(font
+					(size 1.27 1.27)
+				)
+				(hide yes)
+			)
+		)
+		(property "SnapEDA_Link" ""
+			(at 204.47 86.36 0)
 			(effects
 				(font
@@
 			)
 		)
-		(property "MOUSER" ""
+		(property "MOUSER" "603-RC0805FR-074K7L"
+			(at 184.15 97.79 90)
+			(effects
+				(font
+					(size 1.27 1.27)
+				)
+				(hide yes)
+			)
+		)
+		(property "SnapEDA_Link" ""
 			(at 184.15 97.79 90)
 			(effects
@@
 			)
 		)
-		(property "MOUSER" ""
+		(property "MOUSER" "603-RC0805FR-074K7L"
+			(at 92.71 100.33 90)
+			(effects
+				(font
+					(size 1.27 1.27)
+				)
+				(hide yes)
+			)
+		)
+		(property "SnapEDA_Link" ""
 			(at 92.71 100.33 90)
 			(effects
@@
 			)
 		)
-		(property "MOUSER" ""
+		(property "MOUSER" "603-RC0805JR-07100KL"
 			(at 101.6 105.41 90)
+			(effects
+				(font
+					(size 1.27 1.27)
+				)
+				(hide yes)
+			)
+		)
+		(property "SnapEDA_Link" ""
+			(at 101.6 105.41 0)
 			(effects
 				(font
@@
 			)
 		)
-		(property "MOUSER" ""
+		(property "MOUSER" "603-AC0805FR-1047KL"
 			(at 114.3 87.63 90)
+			(effects
+				(font
+					(size 1.27 1.27)
+				)
+				(hide yes)
+			)
+		)
+		(property "SnapEDA_Link" ""
+			(at 114.3 87.63 0)
 			(effects
 				(font
@@
 			)
 		)
+		(property "SnapEDA_Link" ""
+			(at 111.76 100.33 0)
+			(effects
+				(font
+					(size 1.27 1.27)
+				)
+				(hide yes)
+			)
+		)
+		(property "MOUSER" "241-BC847BS_R1_00001"
+			(at 111.76 100.33 0)
+			(effects
+				(font
+					(size 1.27 1.27)
+				)
+				(hide yes)
+			)
+		)
 		(pin "6"
 		)
@@
 			)
 		)
+		(property "SnapEDA_Link" ""
+			(at 201.93 97.79 0)
+			(effects
+				(font
+					(size 1.27 1.27)
+				)
+				(hide yes)
+			)
+		)
+		(property "MOUSER" "241-BC847BS_R1_00001"
+			(at 201.93 97.79 0)
+			(effects
+				(font
+					(size 1.27 1.27)
+				)
+				(hide yes)
+			)
+		)
 		(pin "6"
 		)
@@
 			)
 		)
-		(property "MOUSER" ""
+		(property "MOUSER" "603-RC0805JR-07100KL"
 			(at 193.04 102.87 90)
 			(effects
 				(font
+					(size 1.27 1.27)
+				)
+				(hide yes)
+			)
+		)
+		(property "SnapEDA_Link" ""
+			(at 193.04 102.87 0)
+			(effects
+				(font
