File: FMTransceiver.kicad_pcb (KiCad board)
At the start: 4 copper layers, 100 x 100 mm, 72 parts, among them J101 Conn_Coaxial, J201 Conn_ARM_JTAG_SWD_10, J202 Conn_02x10_Row_Letter_First, Q501 2N7002, Q701 BC847BS, U101 SA818V, U201 STM32U575CITx, U202 CAT24C32, U203 TLV73333PQDBVRQ1, U204 USBLC6-2SC6, U801 LMR51430 500kHz, Y201 8MHz / 20pF

Commit message: chore: migrate <<HASH>> placeholder to <<VERSION>>
Aligns the KiCad title-block placeholder with the new versioning concept
documented at oe5xrx.org/docs/remote-station/hardware/versioning/.

The placeholder is substituted at CI time:
- Release build:  v1.5 → "1.5" (semver only, no `v`, no SHA)
- Debug build:    "BETA-<short-commit>"

No electrical or layout change — pure text replacement on the title-block
silkscreen text. Requires HW-Module-CI feat/version-placeholder
(OE5XRX/HW-Module-CI#4) to be merged first; otherwise CI substitutes
the old <<HASH>> token and leaves the new <<VERSION>> string literal
in the title block until the CI side catches up.

Co-Authored-By: Claude Opus 4.7 <noreply@anthropic.com>
Other:
- board text added: "<<VERSION>>"
- board text removed: "<<HASH>>"
Changed lines of the file:
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@@
 	(title_block
 		(title "FM Module")
-		(rev "<<HASH>>")
+		(rev "<<VERSION>>")
 		(company "Amateurfunkclub für Remote Stationen")
 		(comment 1 "JLC04161H-7628")
@@
 		)
 	)
-	(gr_text "<<HASH>>"
+	(gr_text "<<VERSION>>"
 		(at 153.797 126.695 0)
 		(layer "F.SilkS")
